Commit message: Workaround xacro parsing issue. Revise xacro files

File: robot_specific_config/abb_irb4600_support/urdf/irb4600_60_205.xacro (robot description, xacro)
@@ -1,5 +1,20 @@
 <?xml version="1.0" ?>
 <robot name="abb_irb4600_60_205" xmlns:xacro="http://ros.org/wiki/xacro">
+  <xacro:arg name="use_fake_hardware" default="true"/>
+  <xacro:property name="use_fake_hardware" value="$(arg use_fake_hardware)"/>
+  <xacro:arg name="rws_ip" default="None"/>
+  <xacro:property name="rws_ip" value="$(arg rws_ip)"/>
+  <xacro:arg name="rws_port" default="80"/>
+  <xacro:property name="rws_port" value="$(arg rws_port)"/>
+  <!-- Robot description -->
   <xacro:include filename="$(find abb_irb4600_support)/urdf/irb4600_60_205_macro.xacro"/>
   <xacro:abb_irb4600_60_205 prefix=""/>
+  <!-- ros2_control -->
+  <xacro:include filename="$(find abb_irb4600_support)/urdf/irb4600.ros2_control.xacro" />
+  <xacro:abb_ros2_control
+    name="ABBMultiInterfaceHardware"
+    prefix=""
+    use_fake_hardware="${use_fake_hardware}"
+    rws_ip="${rws_ip}"
+    rws_port="${rws_port}"/>
 </robot>

File: robot_specific_config/abb_irb4600_support/urdf/irb4600_60_205_macro.xacro (robot description, xacro)
@@ -1,4 +1,5 @@
 <?xml version="1.0"?>
 <robot xmlns:xacro="http://ros.org/wiki/xacro">
+  <xacro:include filename="$(find abb_resources)/urdf/common_materials.xacro"/>
   <xacro:macro name="abb_irb4600_60_205" params="prefix">
     <!-- link list -->
@@ -141,5 +142,5 @@
     </joint>
     <!-- end of joint list -->
-    <!-- ROS-Industrial 'base' frame: base_link to ABB World Coordinates transform -->
+    <!-- ROS-Industrial 'base' frame- base_link to ABB World Coordinates transform -->
     <link name="${prefix}base" />
     <joint name="${prefix}base_link-base" type="fixed">
@@ -148,5 +149,5 @@
       <child link="${prefix}base"/>
     </joint>
-    <!-- ROS-Industrial 'flange' frame: attachment point for EEF models -->
+    <!-- ROS-Industrial 'flange' frame- attachment point for EEF models -->
     <link name="${prefix}flange"/>
     <joint type="fixed" name="${prefix}joint_6-flange">
@@ -155,5 +156,5 @@
       <child link="${prefix}flange"/>
     </joint>
-    <!-- ROS-Industrial 'tool0' frame: all-zeros tool frame -->
+    <!-- ROS-Industrial 'tool0' frame- all-zeros tool frame -->
     <link name="${prefix}tool0" />
     <joint name="${prefix}link_6-tool0" type="fixed">
