Commit message: Update materials/colors for each irb4600 robot description xacro

File: robot_specific_config/abb_irb4600_support/urdf/irb4600_20_250.xacro (robot description, xacro)
@@ -1,5 +1,20 @@
 <?xml version="1.0" ?>
 <robot name="abb_irb4600_20_250" xmlns:xacro="http://ros.org/wiki/xacro">
+  <xacro:arg name="use_fake_hardware" default="true"/>
+  <xacro:property name="use_fake_hardware" value="$(arg use_fake_hardware)"/>
+  <xacro:arg name="rws_ip" default="None"/>
+  <xacro:property name="rws_ip" value="$(arg rws_ip)"/>
+  <xacro:arg name="rws_port" default="80"/>
+  <xacro:property name="rws_port" value="$(arg rws_port)"/>
+  <!-- Robot description -->
   <xacro:include filename="$(find abb_irb4600_support)/urdf/irb4600_20_250_macro.xacro"/>
   <xacro:abb_irb4600_20_250 prefix=""/>
+  <!-- ros2_control -->
+  <xacro:include filename="$(find abb_irb4600_support)/urdf/irb4600.ros2_control.xacro" />
+  <xacro:abb_ros2_control
+    name="ABBMultiInterfaceHardware"
+    prefix=""
+    use_fake_hardware="${use_fake_hardware}"
+    rws_ip="${rws_ip}"
+    rws_port="${rws_port}"/>
 </robot>

File: robot_specific_config/abb_irb4600_support/urdf/irb4600_20_250_macro.xacro (robot description, xacro)
@@ -9,5 +9,5 @@
           <mesh filename="package://abb_irb4600_support/meshes/irb4600/collision/base_link.stl"/>
         </geometry>
-        <xacro:material_abb_white/>
+        <xacro:material_abb_yellow />
       </collision>
       <visual name="visual">
@@ -15,8 +15,5 @@
           <mesh filename="package://abb_irb4600_support/meshes/irb4600/visual/base_link.dae"/>
         </geometry>
-        <xacro:material_abb_white/>
-        <material name="yellow">
-          <color rgba="1 1 0 1"/>
-        </material>
+        <xacro:material_abb_graphite_white/>
       </visual>
     </link>
@@ -26,5 +23,5 @@
           <mesh filename="package://abb_irb4600_support/meshes/irb4600/collision/link_1.stl"/>
         </geometry>
-        <xacro:material_abb_white/>
+        <xacro:material_abb_yellow />
       </collision>
       <visual name="visual">
@@ -32,6 +29,5 @@
           <mesh filename="package://abb_irb4600_support/meshes/irb4600/visual/link_1.dae"/>
         </geometry>
-        <xacro:material_abb_white/>
-        <material name="yellow"/>
+        <xacro:material_abb_graphite_white/>
       </visual>
     </link>
@@ -41,5 +37,5 @@
           <mesh filename="package://abb_irb4600_support/meshes/irb4600_20_250/collision/link_2.stl"/>
         </geometry>
-        <xacro:material_abb_white/>
+        <xacro:material_abb_yellow />
       </collision>
       <visual name="visual">
@@ -47,6 +43,5 @@
           <mesh filename="package://abb_irb4600_support/meshes/irb4600_20_250/visual/link_2.dae"/>
         </geometry>
-        <xacro:material_abb_white/>
-        <material name="yellow"/>
+        <xacro:material_abb_graphite_white/>
       </visual>
     </link>
@@ -56,5 +51,5 @@
           <mesh filename="package://abb_irb4600_support/meshes/irb4600_20_250/collision/link_3.stl"/>
         </geometry>
-        <xacro:material_abb_white/>
+        <xacro:material_abb_yellow />
       </collision>
       <visual name="visual">
@@ -62,6 +57,5 @@
           <mesh filename="package://abb_irb4600_support/meshes/irb4600_20_250/visual/link_3.dae"/>
         </geometry>
-        <xacro:material_abb_white/>
-        <material name="yellow"/>
+        <xacro:material_abb_graphite_white/>
       </visual>
     </link>
@@ -71,5 +65,5 @@
           <mesh filename="package://abb_irb4600_support/meshes/irb4600_20_250/collision/link_4.stl"/>
         </geometry>
-        <xacro:material_abb_white/>
+        <xacro:material_abb_yellow />
       </collision>
       <visual name="visual">
@@ -77,6 +71,5 @@
           <mesh filename="package://abb_irb4600_support/meshes/irb4600_20_250/visual/link_4.dae"/>
         </geometry>
-        <xacro:material_abb_white/>
-        <material name="yellow"/>
+        <xacro:material_abb_graphite_white/>
       </visual>
     </link>
@@ -86,5 +79,5 @@
           <mesh filename="package://abb_irb4600_support/meshes/irb4600_20_250/collision/link_5.stl"/>
         </geometry>
-        <xacro:material_abb_white/>
+        <xacro:material_abb_yellow />
       </collision>
       <visual name="visual">
@@ -92,6 +85,5 @@
           <mesh filename="package://abb_irb4600_support/meshes/irb4600_20_250/visual/link_5.dae"/>
         </geometry>
-        <xacro:material_abb_white/>
-        <material name="yellow"/>
+        <xacro:material_abb_graphite_white/>
       </visual>
     </link>
@@ -101,5 +93,5 @@
           <mesh filename="package://abb_irb4600_support/meshes/irb4600_20_250/collision/link_6.stl"/>
         </geometry>
-        <xacro:material_abb_white/>
+        <xacro:material_abb_yellow />
       </collision>
       <visual name="visual">
@@ -107,6 +99,5 @@
           <mesh filename="package://abb_irb4600_support/meshes/irb4600_20_250/visual/link_6.dae"/>
         </geometry>
-        <xacro:material_abb_white/>
-        <material name="yellow"/>
+        <xacro:material_abb_graphite_white/>
       </visual>
     </link>
@@ -156,5 +147,5 @@
     </joint>
     <!-- end of joint list -->
-    <!-- ROS-Industrial 'base' frame: base_link to ABB World Coordinates transform -->
+    <!-- ROS-Industrial 'base' frame- base_link to ABB World Coordinates transform -->
     <link name="${prefix}base" />
     <joint name="${prefix}base_link-base" type="fixed">
@@ -163,5 +154,5 @@
       <child link="${prefix}base"/>
     </joint>
-    <!-- ROS-Industrial 'flange' frame: attachment point for EEF models -->
+    <!-- ROS-Industrial 'flange' frame- attachment point for EEF models -->
     <link name="${prefix}flange"/>
     <joint type="fixed" name="${prefix}joint_6-flange">
@@ -170,5 +161,5 @@
       <child link="${prefix}flange"/>
     </joint>
-    <!-- ROS-Industrial 'tool0' frame: all-zeros tool frame -->
+    <!-- ROS-Industrial 'tool0' frame- all-zeros tool frame -->
     <link name="${prefix}tool0" />
     <joint name="${prefix}link_6-tool0" type="fixed">

File: robot_specific_config/abb_irb4600_support/urdf/irb4600_40_255.xacro (robot description, xacro)
@@ -1,5 +1,20 @@
 <?xml version="1.0" ?>
 <robot name="abb_irb4600_40_255" xmlns:xacro="http://ros.org/wiki/xacro">
+  <xacro:arg name="use_fake_hardware" default="true"/>
+  <xacro:property name="use_fake_hardware" value="$(arg use_fake_hardware)"/>
+  <xacro:arg name="rws_ip" default="None"/>
+  <xacro:property name="rws_ip" value="$(arg rws_ip)"/>
+  <xacro:arg name="rws_port" default="80"/>
+  <xacro:property name="rws_port" value="$(arg rws_port)"/>
+  <!-- Robot description -->
   <xacro:include filename="$(find abb_irb4600_support)/urdf/irb4600_40_255_macro.xacro"/>
   <xacro:abb_irb4600_40_255 prefix=""/>
+  <!-- ros2_control -->
+  <xacro:include filename="$(find abb_irb4600_support)/urdf/irb4600.ros2_control.xacro" />
+  <xacro:abb_ros2_control
+    name="ABBMultiInterfaceHardware"
+    prefix=""
+    use_fake_hardware="${use_fake_hardware}"
+    rws_ip="${rws_ip}"
+    rws_port="${rws_port}"/>
 </robot>

File: robot_specific_config/abb_irb4600_support/urdf/irb4600_40_255_macro.xacro (robot description, xacro)
@@ -9,5 +9,5 @@
           <mesh filename="package://abb_irb4600_support/meshes/irb4600/collision/base_link.stl"/>
         </geometry>
-        <xacro:material_abb_white/>
+        <xacro:material_abb_yellow />
       </collision>
       <visual name="visual">
@@ -15,8 +15,5 @@
           <mesh filename="package://abb_irb4600_support/meshes/irb4600/visual/base_link.dae"/>
         </geometry>
-        <xacro:material_abb_white/>
-        <material name="yellow">
-          <color rgba="1 1 0 1"/>
-        </material>
+        <xacro:material_abb_graphite_white/>
       </visual>
     </link>
@@ -26,5 +23,5 @@
           <mesh filename="package://abb_irb4600_support/meshes/irb4600/collision/link_1.stl"/>
         </geometry>
-        <xacro:material_abb_white/>
+        <xacro:material_abb_yellow />
       </collision>
       <visual name="visual">
@@ -32,6 +29,5 @@
           <mesh filename="package://abb_irb4600_support/meshes/irb4600/visual/link_1.dae"/>
         </geometry>
-        <xacro:material_abb_white/>
-        <material name="yellow"/>
+        <xacro:material_abb_graphite_white/>
       </visual>
     </link>
@@ -41,5 +37,5 @@
           <mesh filename="package://abb_irb4600_support/meshes/irb4600_40_255/collision/link_2.stl"/>
         </geometry>
-        <xacro:material_abb_white/>
+        <xacro:material_abb_yellow />
       </collision>
       <visual name="visual">
@@ -47,6 +43,5 @@
           <mesh filename="package://abb_irb4600_support/meshes/irb4600_40_255/visual/link_2.dae"/>
         </geometry>
-        <xacro:material_abb_white/>
-        <material name="yellow"/>
+        <xacro:material_abb_graphite_white/>
       </visual>
     </link>
@@ -56,5 +51,5 @@
           <mesh filename="package://abb_irb4600_support/meshes/irb4600_40_255/collision/link_3.stl"/>
         </geometry>
-        <xacro:material_abb_white/>
+        <xacro:material_abb_yellow />
       </collision>
       <visual name="visual">
@@ -62,6 +57,5 @@
           <mesh filename="package://abb_irb4600_support/meshes/irb4600_40_255/visual/link_3.dae"/>
         </geometry>
-        <xacro:material_abb_white/>
-        <material name="yellow"/>
+        <xacro:material_abb_graphite_white/>
       </visual>
     </link>
@@ -71,5 +65,5 @@
           <mesh filename="package://abb_irb4600_support/meshes/irb4600_40_255/collision/link_4.stl"/>
         </geometry>
-        <xacro:material_abb_white/>
+        <xacro:material_abb_yellow />
       </collision>
       <visual name="visual">
@@ -77,6 +71,5 @@
           <mesh filename="package://abb_irb4600_support/meshes/irb4600_40_255/visual/link_4.dae"/>
         </geometry>
-        <xacro:material_abb_white/>
-        <material name="yellow"/>
+        <xacro:material_abb_graphite_white/>
       </visual>
     </link>
@@ -86,5 +79,5 @@
           <mesh filename="package://abb_irb4600_support/meshes/irb4600_40_255/collision/link_5.stl"/>
         </geometry>
-        <xacro:material_abb_white/>
+        <xacro:material_abb_yellow />
       </collision>
       <visual name="visual">
@@ -92,6 +85,5 @@
           <mesh filename="package://abb_irb4600_support/meshes/irb4600_40_255/visual/link_5.dae"/>
         </geometry>
-        <xacro:material_abb_white/>
-        <material name="yellow"/>
+        <xacro:material_abb_graphite_white/>
       </visual>
     </link>
@@ -101,5 +93,5 @@
           <mesh filename="package://abb_irb4600_support/meshes/irb4600_40_255/collision/link_6.stl"/>
         </geometry>
-        <xacro:material_abb_white/>
+        <xacro:material_abb_yellow />
       </collision>
       <visual name="visual">
@@ -107,6 +99,5 @@
           <mesh filename="package://abb_irb4600_support/meshes/irb4600_40_255/visual/link_6.dae"/>
         </geometry>
-        <xacro:material_abb_white/>
-        <material name="yellow"/>
+        <xacro:material_abb_graphite_white/>
       </visual>
     </link>
@@ -156,5 +147,5 @@
     </joint>
     <!-- end of joint list -->
-    <!-- ROS-Industrial 'base' frame: base_link to ABB World Coordinates transform -->
+    <!-- ROS-Industrial 'base' frame- base_link to ABB World Coordinates transform -->
     <link name="${prefix}base" />
     <joint name="${prefix}base_link-base" type="fixed">
@@ -163,5 +154,5 @@
       <child link="${prefix}base"/>
     </joint>
-    <!-- ROS-Industrial 'flange' frame: attachment point for EEF models -->
+    <!-- ROS-Industrial 'flange' frame- attachment point for EEF models -->
     <link name="${prefix}flange"/>
     <joint type="fixed" name="${prefix}joint_6-flange">
@@ -170,5 +161,5 @@
       <child link="${prefix}flange"/>
     </joint>
-    <!-- ROS-Industrial 'tool0' frame: all-zeros tool frame -->
+    <!-- ROS-Industrial 'tool0' frame- all-zeros tool frame -->
     <link name="${prefix}tool0" />
     <joint name="${prefix}link_6-tool0" type="fixed">

File: robot_specific_config/abb_irb4600_support/urdf/irb4600_60_205_macro.xacro (robot description, xacro)
@@ -9,4 +9,5 @@
           <mesh filename="package://abb_irb4600_support/meshes/irb4600/collision/base_link.stl"/>
         </geometry>
+        <xacro:material_abb_yellow />
       </collision>
       <visual name="visual">
@@ -14,7 +15,5 @@
           <mesh filename="package://abb_irb4600_support/meshes/irb4600/visual/base_link.dae"/>
         </geometry>
-        <material name="yellow">
-          <color rgba="1 1 0 1"/>
-        </material>
+        <xacro:material_abb_graphite_white/>
       </visual>
     </link>
@@ -24,4 +23,5 @@
           <mesh filename="package://abb_irb4600_support/meshes/irb4600/collision/link_1.stl"/>
         </geometry>
+        <xacro:material_abb_yellow />
       </collision>
       <visual name="visual">
@@ -29,5 +29,5 @@
           <mesh filename="package://abb_irb4600_support/meshes/irb4600/visual/link_1.dae"/>
         </geometry>
-        <material name="yellow"/>
+        <xacro:material_abb_graphite_white/>
       </visual>
     </link>
@@ -37,4 +37,5 @@
           <mesh filename="package://abb_irb4600_support/meshes/irb4600_60_205/collision/link_2.stl"/>
         </geometry>
+        <xacro:material_abb_yellow />
       </collision>
       <visual name="visual">
@@ -42,5 +43,5 @@
           <mesh filename="package://abb_irb4600_support/meshes/irb4600_60_205/visual/link_2.dae"/>
         </geometry>
-        <material name="yellow"/>
+        <xacro:material_abb_graphite_white/>
       </visual>
     </link>
@@ -50,4 +51,5 @@
           <mesh filename="package://abb_irb4600_support/meshes/irb4600_60_205/collision/link_3.stl"/>
         </geometry>
+        <xacro:material_abb_yellow />
       </collision>
       <visual name="visual">
@@ -55,5 +57,5 @@
           <mesh filename="package://abb_irb4600_support/meshes/irb4600_60_205/visual/link_3.dae"/>
         </geometry>
-        <material name="yellow"/>
+        <xacro:material_abb_graphite_white/>
       </visual>
     </link>
@@ -63,4 +65,5 @@
           <mesh filename="package://abb_irb4600_support/meshes/irb4600_60_205/collision/link_4.stl"/>
         </geometry>
+        <xacro:material_abb_yellow />
       </collision>
       <visual name="visual">
@@ -68,5 +71,5 @@
           <mesh filename="package://abb_irb4600_support/meshes/irb4600_60_205/visual/link_4.dae"/>
         </geometry>
-        <material name="yellow"/>
+        <xacro:material_abb_graphite_white/>
       </visual>
     </link>
@@ -76,4 +79,5 @@
           <mesh filename="package://abb_irb4600_support/meshes/irb4600_60_205/collision/link_5.stl"/>
         </geometry>
+        <xacro:material_abb_yellow />
       </collision>
       <visual name="visual">
@@ -81,5 +85,5 @@
           <mesh filename="package://abb_irb4600_support/meshes/irb4600_60_205/visual/link_5.dae"/>
         </geometry>
-        <material name="yellow"/>
+        <xacro:material_abb_graphite_white/>
       </visual>
     </link>
@@ -89,4 +93,5 @@
           <mesh filename="package://abb_irb4600_support/meshes/irb4600_60_205/collision/link_6.stl"/>
         </geometry>
+        <xacro:material_abb_yellow />
       </collision>
       <visual name="visual">
@@ -94,5 +99,5 @@
           <mesh filename="package://abb_irb4600_support/meshes/irb4600_60_205/visual/link_6.dae"/>
         </geometry>
-        <material name="yellow"/>
+        <xacro:material_abb_graphite_white/>
       </visual>
     </link>
