Commit message: add and change files for irb 2600 12 185 version

File: robot_specific_config/abb_irb2600_support/urdf/irb2600_12_185.xacro (robot description, xacro)
@@ -1,5 +1,20 @@
-<?xml version="1.0" encoding="UTF-8"?>
+<?xml version="1.0" ?>
 <robot name="abb_irb2600_12_185" xmlns:xacro="http://ros.org/wiki/xacro">
+  <xacro:arg name="use_fake_hardware" default="true"/>
+  <xacro:property name="use_fake_hardware" value="$(arg use_fake_hardware)"/>
+  <xacro:arg name="rws_ip" default="None"/>
+  <xacro:property name="rws_ip" value="$(arg rws_ip)"/>
+  <xacro:arg name="rws_port" default="80"/>
+  <xacro:property name="rws_port" value="$(arg rws_port)"/>
+  <!-- Robot description -->
   <xacro:include filename="$(find abb_irb2600_support)/urdf/irb2600_12_185_macro.xacro"/>
   <xacro:abb_irb2600_12_185 prefix=""/>
+  <!-- ros2_control -->
+  <xacro:include filename="$(find abb_irb2600_support)/urdf/irb2600.ros2_control.xacro" />
+  <xacro:abb_ros2_control
+    name="ABBMultiInterfaceHardware"
+    prefix=""
+    use_fake_hardware="${use_fake_hardware}"
+    rws_ip="${rws_ip}"
+    rws_port="${rws_port}"/>
 </robot>

File: robot_specific_config/abb_irb2600_support/urdf/irb2600_12_185_macro.xacro (robot description, xacro)
@@ -1,158 +1,158 @@
-<?xml version="1.0" encoding="UTF-8"?>
+<?xml version="1.0"?>
 <robot xmlns:xacro="http://ros.org/wiki/xacro">
   <xacro:include filename="$(find abb_resources)/urdf/common_materials.xacro"/>
   <xacro:macro name="abb_irb2600_12_185" params="prefix">
-    <!-- links -->
+    <!-- link list -->
     <link name="${prefix}base_link">
-      <visual>
-        <origin xyz="0 0 0" rpy="0 0 0" />
+      <collision name="collision">
         <geometry>
-          <mesh filename="package://abb_irb2600_support/meshes/irb2600_12_185/visual/base_link.stl" />
-        </geometry>
-        <xacro:material_abb_orange/>
-      </visual>
-      <collision>
-        <origin xyz="0 0 0" rpy="0 0 0" />
-        <geometry>
-          <mesh filename="package://abb_irb2600_support/meshes/irb2600_12_185/collision/base_link.stl" />
+          <mesh filename="package://abb_irb2600_support/meshes/irb2600_12_185/collision/base_link.stl"/>
         </geometry>
       </collision>
+      <visual name="visual">
+        <geometry>
+          <mesh filename="package://abb_irb2600_support/meshes/irb2600_12_185/visual/base_link.stl"/>
+        </geometry>
+        <xacro:material_abb_yellow />
+      </visual>
     </link>
     <link name="${prefix}link_1">
-      <visual>
-        <origin xyz="0 0 0" rpy="0 0 0" />
+      <collision name="collision">
         <geometry>
-          <mesh filename="package://abb_irb2600_support/meshes/irb2600_12_185/visual/link_1.stl" />
-        </geometry>
-        <xacro:material_abb_orange/>
-      </visual>
-      <collision>
-        <origin xyz="0 0 0" rpy="0 0 0" />
-        <geometry>
-          <mesh filename="package://abb_irb2600_support/meshes/irb2600_12_185/collision/link_1.stl" />
+          <mesh filename="package://abb_irb2600_support/meshes/irb2600_12_185/collision/link_1.stl"/>
         </geometry>
       </collision>
+      <visual name="visual">
+        <geometry>
+          <mesh filename="package://abb_irb2600_support/meshes/irb2600_12_185/visual/link_1.stl"/>
+        </geometry>
+        <xacro:material_abb_yellow />
+      </visual>
     </link>
     <link name="${prefix}link_2">
-      <visual>
-        <origin xyz="-0.15 0 -0.445" rpy="0 0 0" />
+      <collision name="collision">
+      	<origin xyz="-0.15 0 -0.445"/>
         <geometry>
-          <mesh filename="package://abb_irb2600_support/meshes/irb2600_12_185/visual/link_2.stl" />
-        </geometry>
-        <xacro:material_abb_orange/>
-      </visual>
-      <collision>
-        <origin xyz="0 0 0" rpy="0 0 0" />
-        <geometry>
-          <mesh filename="package://abb_irb2600_support/meshes/irb2600_12_185/collision/link_2.stl" />
+          <mesh filename="package://abb_irb2600_support/meshes/irb2600_12_185/collision/link_2.stl"/>
         </geometry>
       </collision>
+      <visual name="visual">
+      	<origin xyz="-0.15 0 -0.445"/>
+        <geometry>
+          <mesh filename="package://abb_irb2600_support/meshes/irb2600_12_185/visual/link_2.stl"/>
+        </geometry>
+        <xacro:material_abb_yellow />
+      </visual>
     </link>
     <link name="${prefix}link_3">
-      <visual>
-        <origin xyz="0 0 0" rpy="0 0 0" />
+      <collision name="collision">
         <geometry>
-          <mesh filename="package://abb_irb2600_support/meshes/irb2600_12_185/visual/link_3.stl" />
-        </geometry>
-        <xacro:material_abb_orange/>
-      </visual>
-      <collision>
-        <origin xyz="0 0 0" rpy="0 0 0" />
-        <geometry>
-          <mesh filename="package://abb_irb2600_support/meshes/irb2600_12_185/collision/link_3.stl" />
+          <mesh filename="package://abb_irb2600_support/meshes/irb2600_12_185/collision/link_3.stl"/>
         </geometry>
       </collision>
+      <visual name="visual">
+        <geometry>
+          <mesh filename="package://abb_irb2600_support/meshes/irb2600_12_185/visual/link_3.stl"/>
+        </geometry>
+        <xacro:material_abb_yellow />
+      </visual>
     </link>
     <link name="${prefix}link_4">
-      <visual>
-        <origin xyz="0 0 0" rpy="0 0 0" />
+      <collision name="collision">
         <geometry>
-          <mesh filename="package://abb_irb2600_support/meshes/irb2600_12_185/visual/link_4.stl" />
-        </geometry>
-        <xacro:material_abb_orange/>
-      </visual>
-      <collision>
-        <origin xyz="0 0 0" rpy="0 0 0" />
-        <geometry>
-          <mesh filename="package://abb_irb2600_support/meshes/irb2600_12_185/collision/link_4.stl" />
+          <mesh filename="package://abb_irb2600_support/meshes/irb2600_12_185/collision/link_4.stl"/>
         </geometry>
       </collision>
+      <visual name="visual">
+        <geometry>
+          <mesh filename="package://abb_irb2600_support/meshes/irb2600_12_185/visual/link_4.stl"/>
+        </geometry>
+        <xacro:material_abb_yellow />
+      </visual>
     </link>
     <link name="${prefix}link_5">
-      <visual>
-        <origin xyz="0 0 0" rpy="0 0 0" />
+      <collision name="collision">
         <geometry>
-          <mesh filename="package://abb_irb2600_support/meshes/irb2600_12_185/visual/link_5.stl" />
-        </geometry>
-        <xacro:material_abb_orange/>
-      </visual>
-      <collision>
-        <origin xyz="0 0 0" rpy="0 0 0" />
-        <geometry>
-          <mesh filename="package://abb_irb2600_support/meshes/irb2600_12_185/collision/link_5.stl" />
+          <mesh filename="package://abb_irb2600_support/meshes/irb2600_12_185/collision/link_5.stl"/>
         </geometry>
       </collision>
+      <visual name="visual">
+        <geometry>
+          <mesh filename="package://abb_irb2600_support/meshes/irb2600_12_185/visual/link_5.stl"/>
+        </geometry>
+        <xacro:material_abb_yellow />
+      </visual>
     </link>
     <link name="${prefix}link_6">
-      <visual>
-        <origin xyz="0 0 0" rpy="0 0 0" />
+      <collision name="collision">
         <geometry>
-          <mesh filename="package://abb_irb2600_support/meshes/irb2600_12_185/visual/link_6.stl" />
-        </geometry>
-        <material name="">
-          <color rgba="0.5 0.5 0.5 1" />
-        </material>
-      </visual>
-      <collision>
-        <origin xyz="0 0 0" rpy="0 0 0" />
-        <geometry>
-          <mesh filename="package://abb_irb2600_support/meshes/irb2600_12_185/collision/link_6.stl" />
+          <mesh filename="package://abb_irb2600_support/meshes/irb2600_12_185/collision/link_6.stl"/>
         </geometry>
       </collision>
+      <visual name="visual">
+        <geometry>
+          <mesh filename="package://abb_irb2600_support/meshes/irb2600_12_185/visual/link_6.stl"/>
+        </geometry>
+        <xacro:material_abb_yellow />
+      </visual>
     </link>
-    <!-- Joints -->
-    <joint name="${prefix}joint_1" type="revolute">
-      <origin xyz="0 0 0.445" rpy="0 0 0" />
-      <parent link="${prefix}base_link" />
-      <child link="${prefix}link_1" />
-      <axis xyz="0 0 1" />
-      <limit lower="-3.14159" upper="3.14159" effort="0" velocity="3.054" />
+    <!-- end of link list -->
+    <!-- joint list -->
+    <joint type="revolute" name="${prefix}joint_1">
+      <origin xyz="0 0 0.445" rpy="0 0 0"/>
+      <axis xyz="0 0 1"/>
+      <parent link="${prefix}base_link"/>
+      <child link="${prefix}link_1"/>
+      <!-- See note 2 in package.xml about effort limits and dynamics values -->
+      <limit lower="-3.14159" upper="3.14159" effort="0" velocity="3.054"/>
+      <dynamics damping="50.0" friction="1.0"/>
     </joint>
-    <joint name="${prefix}joint_2" type="revolute">
-      <origin xyz="0.15 0 0.0" rpy="0 0 0" />
-      <parent link="${prefix}link_1" />
-      <child link="${prefix}link_2" />
-      <axis xyz="0 1 0" />
-      <limit lower="-2.705" upper="1.658" effort="0" velocity="3.054" />
+    <joint type="revolute" name="${prefix}joint_2">
+      <origin xyz="0.15 0 0" rpy="0 0 0"/>
+      <axis xyz="0 1 0"/>
+      <parent link="${prefix}link_1"/>
+      <child link="${prefix}link_2"/>
+      <!-- See note 2 in package.xml about effort limits and dynamics values -->
+      <limit lower="-2.705" upper="1.658" effort="0" velocity="3.054"/>
+      <dynamics damping="50.0" friction="1.0"/>
     </joint>
-    <joint name="${prefix}joint_3" type="revolute">
-      <origin xyz="0 0 0.9" rpy="0 0 0" />
-      <parent link="${prefix}link_2" />
-      <child link="${prefix}link_3" />
-      <axis xyz="0 1 0" />
-      <limit lower="-2.705" upper="1.309" effort="0" velocity="3.054" />
+    <joint type="revolute" name="${prefix}joint_3">
+      <origin xyz="0 0 0.9" rpy="0 0 0"/>
+      <axis xyz="0 1 0"/>
+      <parent link="${prefix}link_2"/>
+      <child link="${prefix}link_3"/>
+      <!-- See note 2 in package.xml about effort limits and dynamics values -->
+      <limit lower="-2.705" upper="1.309" effort="0" velocity="3.054"/>
+      <dynamics damping="10.0" friction="1.0"/>
     </joint>
-    <joint name="${prefix}joint_4" type="revolute">
-      <origin xyz="0 0 0.115" rpy="0 0 0" />
-      <parent link="${prefix}link_3" />
-      <child link="${prefix}link_4" />
-      <axis xyz="1 0 0" />
-      <limit lower="-6.981" upper="6.981" effort="0" velocity="6.283" />
+    <joint type="revolute" name="${prefix}joint_4">
+      <origin xyz="0 0 0.115" rpy="0 0 0"/>
+      <axis xyz="1 0 0"/>
+      <parent link="${prefix}link_3"/>
+      <child link="${prefix}link_4"/>
+      <!-- See note 2 in package.xml about effort limits and dynamics values -->
+      <limit lower="-6.981" upper="6.981" effort="0" velocity="6.283"/>
+      <dynamics damping="5.0" friction="1.0"/>
     </joint>
-    <joint name="${prefix}joint_5" type="revolute">
-      <origin xyz="0.795 0 0 " rpy="0 0 0" />
-      <parent link="${prefix}link_4" />
-      <child link="${prefix}link_5" />
-      <axis xyz="0 1 0" />
-      <limit lower="-2.094" upper="2.094" effort="0" velocity="6.283" />
+    <joint type="revolute" name="${prefix}joint_5">
+      <origin xyz="0.795 0 0" rpy="0 0 0"/>
+      <axis xyz="0 1 0"/>
+      <parent link="${prefix}link_4"/>
+      <child link="${prefix}link_5"/>
+      <!-- See note 2 in package.xml about effort limits and dynamics values -->
+      <limit lower="-2.094" upper="2.094" effort="0" velocity="6.283"/>
+      <dynamics damping="2.0" friction="1.0"/>
     </joint>
-    <joint name="${prefix}joint_6" type="revolute">
-      <origin xyz="0.085 0 0" rpy="0 0 0" />
-      <parent link="${prefix}link_5" />
-      <child link="${prefix}link_6" />
-      <axis xyz="1 0 0" />
-      <limit lower="-6.981" upper="6.981" effort="0" velocity="8.727" />
+    <joint type="revolute" name="${prefix}joint_6">
+      <origin xyz="0.085 0 0" rpy="0 0 0"/>
+      <axis xyz="1 0 0"/>
+      <parent link="${prefix}link_5"/>
+      <child link="${prefix}link_6"/>
+      <!-- See note 2 in package.xml about effort limits and dynamics values -->
+      <limit lower="-6.981" upper="6.981" effort="0" velocity="8.727"/>
+      <dynamics damping="1.0" friction="1.0"/>
     </joint>
-    <!-- ROS-Industrial 'base' frame: base_link to ABB World Coordinates transform -->
+    <!-- end of joint list -->
+    <!-- ROS-Industrial 'base' frame- base_link to ABB World Coordinates transform -->
     <link name="${prefix}base" />
     <joint name="${prefix}base_link-base" type="fixed">
@@ -161,5 +161,5 @@
       <child link="${prefix}base"/>
     </joint>
-    <!-- ROS-Industrial 'flange' frame: attachment point for EEF models -->
+    <!-- ROS-Industrial 'flange' frame- attachment point for EEF models -->
     <link name="${prefix}flange"/>
     <joint type="fixed" name="${prefix}joint_6-flange">
@@ -168,5 +168,5 @@
       <child link="${prefix}flange"/>
     </joint>
-    <!-- ROS-Industrial 'tool0' frame: all-zeros tool frame -->
+    <!-- ROS-Industrial 'tool0' frame- all-zeros tool frame -->
     <link name="${prefix}tool0" />
     <joint name="${prefix}link_6-tool0" type="fixed">
