Commit message: specify correct joint limits

File: robot_specific_config/abb_irb2600_support/urdf/irb2600.ros2_control.xacro (robot description, xacro)
@@ -24,6 +24,6 @@
       <joint name="${prefix}joint_1">
         <command_interface name="position">
-          <param name="min">{-2*pi}</param>
-          <param name="max">{2*pi}</param>
+          <param name="min">-3.142</param>
+          <param name="max">3.142</param>
         </command_interface>
         <command_interface name="velocity"/>
@@ -35,6 +35,6 @@
       <joint name="${prefix}joint_2">
         <command_interface name="position">
-          <param name="min">-2.41</param>
-          <param name="max">2.41</param>
+          <param name="min">-1.658</param>
+          <param name="max">2.705</param>
         </command_interface>
         <command_interface name="velocity"/>
@@ -46,6 +46,6 @@
       <joint name="${prefix}joint_3">
         <command_interface name="position">
-          <param name="min">{-2*pi}</param>
-          <param name="max">{2*pi}</param>
+          <param name="min">-3.142</param>
+          <param name="max">1.309</param>
         </command_interface>
         <command_interface name="velocity"/>
@@ -57,6 +57,6 @@
       <joint name="${prefix}joint_4">
         <command_interface name="position">
-          <param name="min">-2.66</param>
-          <param name="max">2.66</param>
+          <param name="min">-6.981</param>
+          <param name="max">6.981</param>
         </command_interface>
         <command_interface name="velocity"/>
@@ -68,6 +68,6 @@
       <joint name="${prefix}joint_5">
         <command_interface name="position">
-          <param name="min">{-2*pi}</param>
-          <param name="max">{2*pi}</param>
+          <param name="min">-2.094</param>
+          <param name="max">2.094</param>
         </command_interface>
         <command_interface name="velocity"/>
@@ -79,6 +79,6 @@
       <joint name="${prefix}joint_6">
         <command_interface name="position">
-          <param name="min">-2.23</param>
-          <param name="max">2.23</param>
+          <param name="min">-6.981</param>
+          <param name="max">6.981</param>
         </command_interface>
         <command_interface name="velocity"/>

File: robot_specific_config/abb_irb2600_support/urdf/irb2600_12_165_macro.xacro (robot description, xacro)
@@ -117,5 +117,5 @@
       <child link="${prefix}link_1" />
       <axis xyz="0 0 1" />
-      <limit lower="-3.14159" upper="3.14159" effort="0" velocity="3.054" />
+      <limit lower="-3.142" upper="3.142" effort="0" velocity="3.054" />
     </joint>
     <joint name="${prefix}joint_2" type="revolute">
@@ -124,5 +124,5 @@
       <child link="${prefix}link_2" />
       <axis xyz="0 1 0" />
-      <limit lower="-2.705" upper="1.658" effort="0" velocity="3.054" />
+      <limit lower="-1.658" upper="2.705" effort="0" velocity="3.054" />
     </joint>
     <joint name="${prefix}joint_3" type="revolute">
@@ -131,5 +131,5 @@
       <child link="${prefix}link_3" />
       <axis xyz="0 1 0" />
-      <limit lower="-2.705" upper="1.309" effort="0" velocity="3.054" />
+      <limit lower="-3.142" upper="1.309" effort="0" velocity="3.054" />
     </joint>
     <joint name="${prefix}joint_4" type="revolute">

File: robot_specific_config/abb_irb2600_support/urdf/irb2600_12_185_macro.xacro (robot description, xacro)
@@ -105,5 +105,5 @@
       <child link="${prefix}link_1"/>
       <!-- See note 2 in package.xml about effort limits and dynamics values -->
-      <limit lower="-3.14159" upper="3.14159" effort="0" velocity="3.054"/>
+      <limit lower="-3.142" upper="3.142" effort="0" velocity="3.054"/>
       <dynamics damping="50.0" friction="1.0"/>
     </joint>
@@ -114,5 +114,5 @@
       <child link="${prefix}link_2"/>
       <!-- See note 2 in package.xml about effort limits and dynamics values -->
-      <limit lower="-2.705" upper="1.658" effort="0" velocity="3.054"/>
+      <limit lower="-1.658" upper="2.705" effort="0" velocity="3.054"/>
       <dynamics damping="50.0" friction="1.0"/>
     </joint>
@@ -123,5 +123,5 @@
       <child link="${prefix}link_3"/>
       <!-- See note 2 in package.xml about effort limits and dynamics values -->
-      <limit lower="-2.705" upper="1.309" effort="0" velocity="3.054"/>
+      <limit lower="-3.142" upper="1.309" effort="0" velocity="3.054"/>
       <dynamics damping="10.0" friction="1.0"/>
     </joint>
