Commit message: User specifies robotstudio_ip at launch

File: robot_specific_config/abb_irb1200_support/urdf/irb1200.ros2_control.xacro (robot description, xacro)
@@ -1,5 +1,5 @@
 <?xml version="1.0"?>
 <robot xmlns:xacro="http://www.ros.org/wiki/xacro">
-  <xacro:macro name="abb_ros2_control" params="name prefix use_fake_hardware:=true">
+  <xacro:macro name="abb_ros2_control" params="name prefix use_fake_hardware:=true robotstudio_ip">
     <ros2_control name="${name}" type="system">
       <hardware>
@@ -14,5 +14,5 @@
           <plugin>abb_hardware_interface/ABBSystemPositionOnlyHardware</plugin>
           <param name="rws_port">80</param>
-          <param name="rws_ip">127.0.0.1</param>
+          <param name="rws_ip">${robotstudio_ip}</param>
           <param name="rob1egm_port">6511</param>
         </xacro:unless>

File: robot_specific_config/abb_irb1200_support/urdf/irb1200_5_90.xacro (robot description, xacro)
@@ -3,4 +3,6 @@
   <xacro:arg name="use_fake_hardware" default="true"/>
   <xacro:property name="use_fake_hardware" value="$(arg use_fake_hardware)"/>
+  <xacro:arg name="robotstudio_ip" default="None"/>
+  <xacro:property name="robotstudio_ip" value="$(arg robotstudio_ip)"/>
   <!-- Robot description -->
   <xacro:include filename="$(find abb_irb1200_support)/urdf/irb1200_5_90_macro.xacro"/>
@@ -11,4 +13,5 @@
     name="ABBMultiInterfaceHardware"
     prefix=""
-    use_fake_hardware="${use_fake_hardware}"/>
+    use_fake_hardware="${use_fake_hardware}"
+    robotstudio_ip="${robotstudio_ip}"/>
 </robot>

Commit message: Add MultiMove support (#7)
* Switch to using EGMManager

* Each channel needs its own port number, add more comments

* Update abb.repos, hardware parameters, pack and go example, docs

* User specifies robotstudio_ip at launch

* Apply suggestions from code review

File: robot_specific_config/abb_irb1200_support/urdf/irb1200.ros2_control.xacro (robot description, xacro)
@@ -1,5 +1,5 @@
 <?xml version="1.0"?>
 <robot xmlns:xacro="http://www.ros.org/wiki/xacro">
-  <xacro:macro name="abb_ros2_control" params="name prefix use_fake_hardware:=true">
+  <xacro:macro name="abb_ros2_control" params="name prefix use_fake_hardware:=true robotstudio_ip">
     <ros2_control name="${name}" type="system">
       <hardware>
@@ -13,5 +13,7 @@
         <xacro:unless value="${use_fake_hardware}">
           <plugin>abb_hardware_interface/ABBSystemPositionOnlyHardware</plugin>
-          <param name="robotstudio_port">6511</param>
+          <param name="rws_port">80</param>
+          <param name="rws_ip">${robotstudio_ip}</param>
+          <param name="rob1egm_port">6511</param>
         </xacro:unless>
       </hardware>

Commit message: Make rws_port configurable from launch

File: robot_specific_config/abb_irb1200_support/urdf/irb1200.ros2_control.xacro (robot description, xacro)
@@ -1,5 +1,5 @@
 <?xml version="1.0"?>
 <robot xmlns:xacro="http://www.ros.org/wiki/xacro">
-  <xacro:macro name="abb_ros2_control" params="name prefix use_fake_hardware:=true robotstudio_ip">
+  <xacro:macro name="abb_ros2_control" params="name prefix use_fake_hardware:=true rws_ip rws_port">
     <ros2_control name="${name}" type="system">
       <hardware>
@@ -13,6 +13,6 @@
         <xacro:unless value="${use_fake_hardware}">
           <plugin>abb_hardware_interface/ABBSystemPositionOnlyHardware</plugin>
-          <param name="rws_port">80</param>
-          <param name="rws_ip">${robotstudio_ip}</param>
+          <param name="rws_port">${rws_port}</param>
+          <param name="rws_ip">${rws_ip}</param>
           <!-- The following parameter is used for the non-MultiMove only -->
           <param name="egm_port">6511</param>

File: robot_specific_config/abb_irb1200_support/urdf/irb1200_5_90.xacro (robot description, xacro)
@@ -3,6 +3,8 @@
   <xacro:arg name="use_fake_hardware" default="true"/>
   <xacro:property name="use_fake_hardware" value="$(arg use_fake_hardware)"/>
-  <xacro:arg name="robotstudio_ip" default="None"/>
-  <xacro:property name="robotstudio_ip" value="$(arg robotstudio_ip)"/>
+  <xacro:arg name="rws_ip" default="None"/>
+  <xacro:property name="rws_ip" value="$(arg rws_ip)"/>
+  <xacro:arg name="rws_port" default="80"/>
+  <xacro:property name="rws_port" value="$(arg rws_port)"/>
   <!-- Robot description -->
   <xacro:include filename="$(find abb_irb1200_support)/urdf/irb1200_5_90_macro.xacro"/>
@@ -14,4 +16,5 @@
     prefix=""
     use_fake_hardware="${use_fake_hardware}"
-    robotstudio_ip="${robotstudio_ip}"/>
+    rws_ip="${rws_ip}"
+    rws_port="${rws_port}"/>
 </robot>

Commit message: Generate robot controller description from ros2_control xacro
Signed-off-by: Yadunund <yadunund@openrobotics.org>

File: robot_specific_config/abb_irb1200_support/urdf/irb1200.ros2_control.xacro (robot description, xacro)
@@ -1,5 +1,5 @@
 <?xml version="1.0"?>
 <robot xmlns:xacro="http://www.ros.org/wiki/xacro">
-  <xacro:macro name="abb_ros2_control" params="name prefix use_fake_hardware:=true rws_ip rws_port">
+  <xacro:macro name="abb_ros2_control" params="name prefix use_fake_hardware:=true rws_ip rws_port configure_via_rws:=true">
     <ros2_control name="${name}" type="system">
       <hardware>
@@ -13,4 +13,9 @@
         <xacro:unless value="${use_fake_hardware}">
           <plugin>abb_hardware_interface/ABBSystemHardware</plugin>
+          <!-- If false, the robot description required for EGM connection-->
+          <!-- will be generated as per joint information listed below. -->
+          <!-- If true, the robot description will be generated by retrieving -->
+          <!-- information from the ABB controller via RWS. -->
+          <param name="configure_via_rws">${configure_via_rws}</param>
           <param name="rws_port">${rws_port}</param>
           <param name="rws_ip">${rws_ip}</param>
@@ -24,6 +29,6 @@
       <joint name="${prefix}joint_1">
         <command_interface name="position">
-          <param name="min">{-2*pi}</param>
-          <param name="max">{2*pi}</param>
+          <param name="min">${-2*pi}</param>
+          <param name="max">${2*pi}</param>
         </command_interface>
         <command_interface name="velocity"/>
@@ -46,6 +51,6 @@
       <joint name="${prefix}joint_3">
         <command_interface name="position">
-          <param name="min">{-2*pi}</param>
-          <param name="max">{2*pi}</param>
+          <param name="min">${-2*pi}</param>
+          <param name="max">${2*pi}</param>
         </command_interface>
         <command_interface name="velocity"/>
@@ -68,6 +73,6 @@
       <joint name="${prefix}joint_5">
         <command_interface name="position">
-          <param name="min">{-2*pi}</param>
-          <param name="max">{2*pi}</param>
+          <param name="min">${-2*pi}</param>
+          <param name="max">${2*pi}</param>
         </command_interface>
         <command_interface name="velocity"/>

File: robot_specific_config/abb_irb1200_support/urdf/irb1200_5_90.xacro (robot description, xacro)
@@ -7,4 +7,6 @@
   <xacro:arg name="rws_port" default="80"/>
   <xacro:property name="rws_port" value="$(arg rws_port)"/>
+  <xacro:arg name="configure_via_rws" default="true"/>
+  <xacro:property name="configure_via_rws" value="$(arg configure_via_rws)"/>
   <!-- Robot description -->
   <xacro:include filename="$(find abb_irb1200_support)/urdf/irb1200_5_90_macro.xacro"/>
@@ -17,4 +19,5 @@
     use_fake_hardware="${use_fake_hardware}"
     rws_ip="${rws_ip}"
-    rws_port="${rws_port}"/>
+    rws_port="${rws_port}"
+    configure_via_rws="${configure_via_rws}"/>
 </robot>
