Commit message: Support Omnicore controllers (#56)
* Generate robot controller description from ros2_control xacro

Signed-off-by: Yadunund <yadunund@openrobotics.org>

* Wrap description as string parameter

Signed-off-by: Yadunund <yadunund@openrobotics.org>

* Remove choices arg for launch parameters

Signed-off-by: Yadunund <yadunund@openrobotics.org>

* Cleanup moveit_config

Signed-off-by: Yadunund <yadunund@openrobotics.org>

* Remove newline

Signed-off-by: Yadunund <yadunund@openrobotics.org>

---------

Signed-off-by: Yadunund <yadunund@openrobotics.org>

File: robot_specific_config/abb_irb1200_support/urdf/irb1200_5_90.xacro (robot description, xacro)
@@ -7,4 +7,6 @@
   <xacro:arg name="rws_port" default="80"/>
   <xacro:property name="rws_port" value="$(arg rws_port)"/>
+  <xacro:arg name="configure_via_rws" default="true"/>
+  <xacro:property name="configure_via_rws" value="$(arg configure_via_rws)"/>
   <!-- Robot description -->
   <xacro:include filename="$(find abb_irb1200_support)/urdf/irb1200_5_90_macro.xacro"/>
@@ -17,4 +19,5 @@
     use_fake_hardware="${use_fake_hardware}"
     rws_ip="${rws_ip}"
-    rws_port="${rws_port}"/>
+    rws_port="${rws_port}"
+    configure_via_rws="${configure_via_rws}"/>
 </robot>
