Commit message: add irb6640 supprt to abb_ros2 package

File: robot_specific_config/abb_irb6640_support/urdf/irb6640_185_280.urdf.xacro (robot description, xacro)
@@ -10,10 +10,7 @@
   <xacro:include filename="$(find abb_irb6640_support)/urdf/irb6640_185_280/irb6640_185_280_macro.xacro"/>
   <xacro:include filename="$(find abb_irb6640_support)/urdf/irb6640_185_280/irb6640_185_280_macro.ros2_control.xacro"/>
-  <!-- create link fixed to the "world" -->
-  <link name="world" />
   <!-- Load robot's macro with parameters -->
   <!-- set prefix if multiple robots are used -->
-  <xacro:irb6640_185_280 prefix="$(arg prefix)" parent="world" >
-    <origin xyz="0 0 0" rpy="0 0 0" />          <!-- position robot in the world -->
+  <xacro:irb6640_185_280 prefix="$(arg prefix)" >
   </xacro:irb6640_185_280>
   <xacro:irb6640_185_280_ros2_control

File: robot_specific_config/abb_irb6640_support/urdf/irb6640_185_280/irb6640_185_280_macro.ros2_control.xacro (robot description, xacro)
@@ -26,5 +26,5 @@
         </xacro:unless>
       </hardware>
-      <joint name="${prefix}joint1">
+      <joint name="${prefix}joint_1">
         <command_interface name="position">     <!-- Add/Remove interfaces as needed -->
           <param name="min">-1</param>
@@ -37,5 +37,5 @@
         <state_interface name="acceleration"/>
       </joint>
-      <joint name="${prefix}joint2">
+      <joint name="${prefix}joint_2">
         <command_interface name="position">     <!-- Add/Remove interfaces as needed -->
           <param name="min">-1</param>
@@ -48,5 +48,5 @@
         <state_interface name="acceleration"/>
       </joint>
-      <joint name="${prefix}joint3">
+      <joint name="${prefix}joint_3">
         <command_interface name="position">     <!-- Add/Remove interfaces as needed -->
           <param name="min">-1</param>
@@ -59,5 +59,5 @@
         <state_interface name="acceleration"/>
       </joint>
-      <joint name="${prefix}joint4">
+      <joint name="${prefix}joint_4">
         <command_interface name="position">     <!-- Add/Remove interfaces as needed -->
           <param name="min">-1</param>
@@ -70,5 +70,5 @@
         <state_interface name="acceleration"/>
       </joint>
-      <joint name="${prefix}joint5">
+      <joint name="${prefix}joint_5">
         <command_interface name="position">     <!-- Add/Remove interfaces as needed -->
           <param name="min">-1</param>
@@ -81,5 +81,5 @@
         <state_interface name="acceleration"/>
       </joint>
-      <joint name="${prefix}joint6">
+      <joint name="${prefix}joint_6">
         <command_interface name="position">     <!-- Add/Remove interfaces as needed -->
           <param name="min">-1</param>
@@ -92,25 +92,4 @@
         <state_interface name="acceleration"/>
       </joint>
-      <sensor name="tcp_fts_sensor">            <!-- Remove/change sensors as needed -->
-        <state_interface name="fx"/>
-        <state_interface name="fy"/>
-        <state_interface name="fz"/>
-        <state_interface name="tx"/>
-        <state_interface name="ty"/>
-        <state_interface name="tz"/>
-        <param name="frame_id">tool0</param>    <!-- Change sensors as needed -->
-        <param name="min_fx">-100</param>
-        <param name="max_fx">100</param>
-        <param name="min_fy">-100</param>
-        <param name="max_fy">100</param>
-        <param name="min_fz">-200</param>
-        <param name="max_fz">200</param>
-        <param name="min_tx">-10</param>
-        <param name="max_tx">10</param>
-        <param name="min_ty">-10</param>
-        <param name="max_ty">10</param>
-        <param name="min_tz">-15</param>
-        <param name="max_tz">15</param>
-      </sensor>
     </ros2_control>
     <xacro:if value="$(arg sim_gazebo_classic)">

File: robot_specific_config/abb_irb6640_support/urdf/irb6640_185_280/irb6640_185_280_macro.xacro (robot description, xacro)
@@ -1,235 +1,200 @@
 <?xml version="1.0" encoding="UTF-8"?>
 <robot xmlns:xacro="http://wiki.ros.org/xacro">
-  <xacro:include filename="$(find abb_irb6640_support)/urdf/common.xacro" />
-  <xacro:macro name="irb6640_185_280" params="prefix parent *origin">
-    <!-- LINKS -->
-    <!-- base link -->
+  <xacro:macro name="irb6640_185_280" params="prefix">
+    <xacro:include filename="$(find abb_resources)/urdf/common_materials.xacro"/>
+    <xacro:include filename="$(find abb_resources)/urdf/inertials.xacro"/>
+    <!-- link list -->
     <link name="${prefix}base_link">
-      <!-- Default inertial for Gazebo/Ingnition - copy and edit block from 'common.xacro'
-           to get more realistic behaviour-->
-      <xacro:default_inertial/>
-      <visual>
-        <origin xyz="0 0 0" rpy="0 0 0" />
-        <geometry>
-          <cylinder length="0.3" radius="0.3" />
-<!--           <mesh filename="package://abb_irb6640_support/meshes/irb6640_185_280/visual/base_link.dae" /> -->
-        </geometry>
-      </visual>
-      <collision>
-        <origin xyz="0 0 0" rpy="0 0 0" />
-        <geometry>
-          <cylinder length="0.3" radius="0.3" />
-<!--           <mesh filename="package://abb_irb6640_support/meshes/irb6640_185_280/collision/base_link.stl" /> -->
-        </geometry>
-      </collision>
-    </link>
-    <!-- link 1 -->
-    <link name="${prefix}link1">
-      <!-- Default inertial for Gazebo/Ingnition - copy and edit block from 'common.xacro'
-           to get more realistic behaviour-->
-      <xacro:default_inertial/>
-      <visual>
-        <origin xyz="0 0 0" rpy="0 0 0" />
-        <geometry>
-          <cylinder length="0.3" radius="0.15" />
-<!--           <mesh filename="package://abb_irb6640_support/meshes/irb6640_185_280/visual/link1.dae" /> -->
-        </geometry>
-      </visual>
-      <collision>
-        <origin xyz="0 0 0" rpy="0 0 0" />
-        <geometry>
-          <cylinder length="0.3" radius="0.15" />
-<!--           <mesh filename="package://abb_irb6640_support/meshes/irb6640_185_280/collision/link1.stl" /> -->
-        </geometry>
-      </collision>
-    </link>
-    <!-- link 2 -->
-    <link name="${prefix}link2">
-      <!-- Default inertial for Gazebo/Ingnition - copy and edit block from 'common.xacro'
-           to get more realistic behaviour-->
-      <xacro:default_inertial/>
-      <visual>
-        <origin xyz="0 0 0" rpy="0 0 0" />
-        <geometry>
-          <cylinder length="0.8" radius="0.15" />
-<!--           <mesh filename="package://abb_irb6640_support/meshes/irb6640_185_280/visual/link2.dae" /> -->
-        </geometry>
-      </visual>
-      <collision>
-        <origin xyz="0 0 0" rpy="0 0 0" />
-        <geometry>
-          <cylinder length="0.8" radius="0.15" />
-<!--           <mesh filename="package://abb_irb6640_support/meshes/irb6640_185_280/collision/link2.stl"  /> -->
-        </geometry>
-      </collision>
-    </link>
-    <!-- link 3 -->
-    <link name="${prefix}link3">
-      <!-- Default inertial for Gazebo/Ingnition - copy and edit block from 'common.xacro'
-           to get more realistic behaviour-->
-      <xacro:default_inertial/>
-      <visual>
-        <origin xyz="0 0 0" rpy="0 0 0" />
-        <geometry>
-          <cylinder length="0.5" radius="0.10" />
-<!--           <mesh filename="package://abb_irb6640_support/meshes/irb6640_185_280/visual/link3.dae" /> -->
-        </geometry>
-      </visual>
-      <collision>
-        <origin xyz="0 0 0" rpy="0 0 0" />
-        <geometry>
-          <cylinder length="0.5" radius="0.10" />
-<!--           <mesh filename="package://abb_irb6640_support/meshes/irb6640_185_280/collision/link3.stl"  /> -->
-        </geometry>
-      </collision>
-    </link>
-    <!-- link 4 -->
-    <link name="${prefix}link4">
-      <!-- Default inertial for Gazebo/Ingnition - copy and edit block from 'common.xacro'
-           to get more realistic behaviour-->
-      <xacro:default_inertial/>
-      <visual>
-        <origin xyz="0 0 0" rpy="0 0 0" />
-        <geometry>
-          <cylinder length="0.1" radius="0.2" />
-<!--           <mesh filename="package://abb_irb6640_support/meshes/irb6640_185_280/visual/link4.dae" /> -->
-        </geometry>
-      </visual>
-      <collision>
-        <origin xyz="0 0 0" rpy="0 0 0" />
-        <geometry>
-          <cylinder length="0.1" radius="0.2" />
-<!--           <mesh filename="package://abb_irb6640_support/meshes/irb6640_185_280/collision/link4.stl"  /> -->
-        </geometry>
-      </collision>
-    </link>
-    <!-- link 5 -->
-    <link name="${prefix}link5">
-      <!-- Default inertial for Gazebo/Ingnition - copy and edit block from 'common.xacro'
-           to get more realistic behaviour-->
-      <xacro:default_inertial/>
-      <visual>
-        <origin xyz="0 0 0" rpy="0 0 0" />
-        <geometry>
-          <cylinder length="0.2" radius="0.1" />
-<!--           <mesh filename="package://abb_irb6640_support/meshes/irb6640_185_280/visual/link5.dae" /> -->
-        </geometry>
-      </visual>
-      <collision>
-        <origin xyz="0 0 0" rpy="0 0 0" />
-        <geometry>
-          <cylinder length="0.2" radius="0.1" />
-<!--           <mesh filename="package://abb_irb6640_support/meshes/irb6640_185_280/collision/link5.stl" /> -->
-        </geometry>
-      </collision>
-    </link>
-    <!-- link 6 -->
-    <link name="${prefix}link6">
-      <!-- Default inertial for Gazebo/Ingnition - copy and edit block from 'common.xacro'
-           to get more realistic behaviour-->
-      <xacro:default_inertial/>
-      <visual>
-        <origin xyz="0 0 0" rpy="0 0 0" />
-        <geometry>
-          <cylinder length="0.05" radius="0.1" />
-<!--           <mesh filename="package://abb_irb6640_support/meshes/irb6640_185_280/visual/link6.dae" /> -->
-        </geometry>
-      </visual>
-      <collision>
-        <origin xyz="0 0 0" rpy="0 0 0" />
-        <geometry>
-          <cylinder length="0.05" radius="0.1" />
-<!--           <mesh filename="package://abb_irb6640_support/meshes/irb6640_185_280/collision/link6.stl" /> -->
-        </geometry>
-      </collision>
-    </link>
-    <!-- All-zero tool frame. This frame should correspond to the TOOL frame of the robot's controller.) -->
-    <link name="${prefix}tool0" />
-    <!-- tool link -->
-<!-- START Delete if not needed -->
-    <!-- Standard frames for industrial robots. Also useful for manipulators.
-         (ROS-I specs - https://wiki.ros.org/Industrial/Tutorials/WorkingWithRosIndustrialRobotSupportPackages#Standardised_links_.2F_frames)-->
-    <!-- This frame should correspond to the BASE coordinate system of robot's controller.) -->
+      <collision name="collision">
+        <geometry>
+          <mesh filename="package://abb_irb6640_support/meshes/irb6640_185_280/collision/base_link.stl"/>
+        </geometry>
+      </collision>
+      <visual name="visual">
+        <geometry>
+          <mesh filename="package://abb_irb6640_support/meshes/irb6640_185_280/visual/base_link.dae"/>
+        </geometry>
+        <material name="yellow">
+          <color rgba="1 1 0 1"/>
+        </material>
+      </visual>
+    </link>
+    <link name="${prefix}link_1">
+      <collision name="collision">
+        <geometry>
+          <mesh filename="package://abb_irb6640_support/meshes/irb6640_185_280/collision/link_1.stl"/>
+        </geometry>
+      </collision>
+      <visual name="visual">
+        <geometry>
+          <mesh filename="package://abb_irb6640_support/meshes/irb6640_185_280/visual/link_1.dae"/>
+        </geometry>
+        <material name="yellow"/>
+      </visual>
+    </link>
+    <link name="${prefix}link_2">
+      <collision name="collision">
+        <geometry>
+          <mesh filename="package://abb_irb6640_support/meshes/irb6640_185_280/collision/link_2.stl"/>
+        </geometry>
+      </collision>
+      <visual name="visual">
+        <geometry>
+          <mesh filename="package://abb_irb6640_support/meshes/irb6640_185_280/visual/link_2.dae"/>
+        </geometry>
+        <material name="yellow"/>
+      </visual>
+    </link>
+    <link name="${prefix}link_3">
+      <collision name="collision">
+        <geometry>
+          <mesh filename="package://abb_irb6640_support/meshes/irb6640_185_280/collision/link_3.stl"/>
+        </geometry>
+      </collision>
+      <visual name="visual">
+        <geometry>
+          <mesh filename="package://abb_irb6640_support/meshes/irb6640_185_280/visual/link_3.dae"/>
+        </geometry>
+        <material name="yellow"/>
+      </visual>
+    </link>
+    <link name="${prefix}link_4">
+      <collision name="collision">
+        <geometry>
+          <mesh filename="package://abb_irb6640_support/meshes/irb6640_185_280/collision/link_4.stl"/>
+        </geometry>
+      </collision>
+      <visual name="visual">
+        <geometry>
+          <mesh filename="package://abb_irb6640_support/meshes/irb6640_185_280/visual/link_4.dae"/>
+        </geometry>
+        <material name="yellow"/>
+      </visual>
+    </link>
+    <link name="${prefix}link_5">
+      <collision name="collision">
+        <geometry>
+          <mesh filename="package://abb_irb6640_support/meshes/irb6640_185_280/collision/link_5.stl"/>
+        </geometry>
+      </collision>
+      <visual name="visual">
+        <geometry>
+          <mesh filename="package://abb_irb6640_support/meshes/irb6640_185_280/visual/link_5.dae"/>
+        </geometry>
+        <material name="yellow"/>
+      </visual>
+    </link>
+    <link name="${prefix}link_6">
+      <collision name="collision">
+        <geometry>
+          <mesh filename="package://abb_irb6640_support/meshes/irb6640_185_280/collision/link_6.stl"/>
+        </geometry>
+      </collision>
+      <visual name="visual">
+        <geometry>
+          <mesh filename="package://abb_irb6640_support/meshes/irb6640_185_280/visual/link_6.dae"/>
+        </geometry>
+        <material name="yellow"/>
+      </visual>
+    </link>
+    <link name="${prefix}tool0"/>
+    <!--Cylinder and piston -->
+    <link name="${prefix}link_cylinder">
+      <collision name="collision">
+        <geometry>
+          <mesh filename="package://abb_irb6640_support/meshes/irb6640_185_280/collision/cylinder_link.stl"/>
+        </geometry>
+      </collision>
+      <visual name="visual">
+        <geometry>
+          <mesh filename="package://abb_irb6640_support/meshes/irb6640_185_280/visual/cylinder_link.dae"/>
+        </geometry>
+        <material name="yellow"/>
+      </visual>
+    </link>
+    <link name="${prefix}link_piston">
+      <collision name="collision">
+        <geometry>
+          <mesh filename="package://abb_irb6640_support/meshes/irb6640_185_280/collision/piston_link.stl"/>
+        </geometry>
+      </collision>
+      <visual name="visual">
+        <geometry>
+          <mesh filename="package://abb_irb6640_support/meshes/irb6640_185_280/visual/piston_link.dae"/>
+        </geometry>
+        <material name="yellow"/>
+      </visual>
+    </link>
+    <!-- end of link list -->
+    <!-- joint list -->
+    <joint type="revolute" name="${prefix}joint_1">
+      <origin xyz="0 0 0.780" rpy="0 0 0"/>
+      <axis xyz="0 0 1"/>
+      <parent link="${prefix}base_link"/>
+      <child link="${prefix}link_1"/>
+      <limit effort="0" lower="-2.967" upper="2.967" velocity="1.7453"/>
+    </joint>
+    <joint type="revolute" name="${prefix}joint_2">
+      <origin xyz="0.320 0 0" rpy="0 0 0"/>
+      <axis xyz="0 1 0"/>
+      <parent link="${prefix}link_1"/>
+      <child link="${prefix}link_2"/>
+      <limit effort="0" lower="-1.134" upper="1.4855" velocity="1.5707"/>
+    </joint>
+    <joint type="revolute" name="${prefix}joint_3">
+      <origin xyz="0 0 1.075" rpy="0 0 0"/>
+      <axis xyz="0 1 0"/>
+      <parent link="${prefix}link_2"/>
+      <child link="${prefix}link_3"/>
+      <limit effort="0" lower="-3.142" upper="1.222" velocity="1.5707"/>
+    </joint>
+    <joint type="revolute" name="${prefix}joint_4">
+      <origin xyz="0 0 0.2" rpy="0 0 0"/>
+      <axis xyz="1 0 0"/>
+      <parent link="${prefix}link_3"/>
+      <child link="${prefix}link_4"/>
+      <limit effort="0" lower="-5.236" upper="5.236" velocity="2.9671"/>
+    </joint>
+    <joint type="revolute" name="${prefix}joint_5">
+      <origin xyz="1.392 0 0 " rpy="0 0 0"/>
+      <axis xyz="0 1 0"/>
+      <parent link="${prefix}link_4"/>
+      <child link="${prefix}link_5"/>
+      <limit effort="0" lower="-2.094" upper="2.094" velocity="2.4435"/>
+    </joint>
+    <joint type="revolute" name="${prefix}joint_6">
+      <origin xyz="0.2 0 0 " rpy="0 0 0"/>
+      <axis xyz="1 0 0"/>
+      <parent link="${prefix}link_5"/>
+      <child link="${prefix}link_6"/>
+      <limit effort="0" lower="-6.283" upper="6.283" velocity="3.3161"/>
+    </joint>
+    <joint type="fixed" name="${prefix}joint_6-tool0">
+      <parent link="${prefix}link_6"/>
+      <child link="${prefix}tool0"/>
+      <origin xyz="0 0 0" rpy="0 1.57079632679 0"/>
+    </joint>
+    <joint type="continuous" name="${prefix}joint_cylinder">
+      <origin xyz="-0.3647 0 -0.1455" rpy="0 0 0"/>
+      <axis xyz="0 1 0"/>
+      <parent link="${prefix}link_1"/>
+      <child link="${prefix}link_cylinder"/>
+      <mimic joint="${prefix}joint_2" multiplier="-0.25"/>
+    </joint>
+    <joint type="continuous" name="${prefix}joint_piston">
+      <origin xyz="-0.22 0 -0.0672" rpy="0 0 0"/>
+      <axis xyz="0 1 0"/>
+      <parent link="${prefix}link_2"/>
+      <child link="${prefix}link_piston"/>
+      <mimic joint="${prefix}joint_2" multiplier="-1.25"/>
+    </joint>
+    <!-- end of joint list -->
+    <!-- ROS base_link to ABB World Coordinates transform -->
     <link name="${prefix}base" />
-    <!-- Frame for mounting EEF models to a manipulator. x+ axis points forward (REP 103). -->
-    <link name="${prefix}flange" />
-<!-- END Delete if not needed  -->
-    <!-- END LINKS -->
-    <!-- JOINTS -->
-    <!-- base_joint fixes base_link to the environment -->
-    <joint name="${prefix}base_joint" type="fixed">
-      <xacro:insert_block name="origin" />
-      <parent link="${parent}" />
-      <child link="${prefix}base_link" />
-    </joint>
-    <!-- joint 1 -->
-    <joint name="${prefix}joint1" type="revolute">
-      <origin xyz="0 0 0.3" rpy="${pi} 0 0" />
-      <parent link="${prefix}base_link" />
-      <child link="${prefix}link1" />
-      <axis xyz="0 0 1" />
-      <limit effort="0" lower="${radians(-180)}" upper="${radians(180)}" velocity="${radians(180)}" />
-    </joint>
-    <!-- joint 2 -->
-    <joint name="${prefix}joint2" type="revolute">
-      <origin xyz="0 0 0.3" rpy="${pi/2} 0 0" />
-      <parent link="${prefix}link1" />
-      <child link="${prefix}link2" />
-      <axis xyz="0 0 1" />
-      <limit effort="0" lower="${radians(-180)}" upper="${radians(180)}" velocity="${radians(180)}" />
-    </joint>
-    <!-- joint 3 -->
-    <joint name="${prefix}joint3" type="revolute">
-      <origin xyz="0.8 0 0" rpy="0 0 0" />
-      <parent link="${prefix}link2" />
-      <child link="${prefix}link3" />
-      <axis xyz="0 0 1" />
-      <limit effort="0" lower="${radians(-90)}" upper="${radians(180)}" velocity="${radians(270)}" />
-    </joint>
-    <!-- joint 4 -->
-    <joint name="${prefix}joint4" type="revolute">
-      <origin xyz="0 0.1 0" rpy="0 ${-pi/2} 0" />
-      <parent link="${prefix}link3" />
-      <child link="${prefix}link4" />
-      <axis xyz="0 0 1" />
-      <limit effort="0" lower="${radians(-360)}" upper="${radians(360)}" velocity="${radians(360)}" />
-    </joint>
-    <!-- joint 5 -->
-    <joint name="${prefix}joint5" type="revolute">
-      <origin xyz="0 0 -0.1" rpy="0 ${pi/2} 0" />
-      <parent link="${prefix}link4" />
-      <child link="${prefix}link5" />
-      <axis xyz="0 0 1" />
-      <limit effort="0" lower="${radians(-120)}" upper="${radians(120)}" velocity="${radians(540)}" />
-    </joint>
-    <!-- joint 6 -->
-    <joint name="${prefix}joint6" type="revolute">
-      <origin xyz="0 0 0.1" rpy="0 ${-pi/2} 0" />
-      <parent link="${prefix}link5" />
-      <child link="${prefix}link6" />
-      <axis xyz="0 0 1" />
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