Commit message: declared piston_joint and cylinder_joint as mimic joints

File: robot_specific_config/abb_irb6640_support/urdf/irb6640_205/irb6640_205_macro.ros2_control.xacro (robot description, xacro)
@@ -92,4 +92,17 @@
         <state_interface name="acceleration"/>
       </joint>
+      <!-- Mimic joints -->
+      <joint name="${prefix}piston_joint">
+        <param name="mimic">joint2</param>
+        <param name="multiplier">-1.3</param>
+        <command_interface name="position"/>
+        <state_interface name="position"/>
+      </joint>
+      <joint name="${prefix}cylinder_joint">
+        <param name="mimic">joint1</param>
+        <param name="multiplier">-0.3</param>
+        <command_interface name="position"/>
+        <state_interface name="position"/>
+      </joint>
     </ros2_control>
     <xacro:if value="$(arg sim_gazebo_classic)">
