Commit message: Reorder control joints to match chain

File: robot_specific_config/abb_irb14000_support/urdf/irb14000_ros2_control.xacro (robot description, xacro)
@@ -35,4 +35,14 @@
         <state_interface name="position">
           <param name="initial_value">${radians(-130)}</param>
+        </state_interface>
+        <state_interface name="velocity">
+          <param name="initial_value">0.0</param>
+        </state_interface>
+      </joint>
+      <joint name="${prefix}robl_joint_7">
+        <command_interface name="position" />
+        <command_interface name="velocity" />
+        <state_interface name="position">
+          <param name="initial_value">${radians(135)}</param>
         </state_interface>
         <state_interface name="velocity">
@@ -80,14 +90,4 @@
         </state_interface>
       </joint>
-      <joint name="${prefix}robl_joint_7">
-        <command_interface name="position" />
-        <command_interface name="velocity" />
-        <state_interface name="position">
-          <param name="initial_value">${radians(135)}</param>
-        </state_interface>
-        <state_interface name="velocity">
-          <param name="initial_value">0.0</param>
-        </state_interface>
-      </joint>
       <joint name="${prefix}robr_joint_1">
         <command_interface name="position" />
@@ -105,4 +105,14 @@
         <state_interface name="position">
           <param name="initial_value">${radians(-130)}</param>
+        </state_interface>
+        <state_interface name="velocity">
+          <param name="initial_value">0.0</param>
+        </state_interface>
+      </joint>
+      <joint name="${prefix}robr_joint_7">
+        <command_interface name="position" />
+        <command_interface name="velocity" />
+        <state_interface name="position">
+          <param name="initial_value">${radians(-135)}</param>
         </state_interface>
         <state_interface name="velocity">
@@ -150,14 +160,4 @@
         </state_interface>
       </joint>
-      <joint name="${prefix}robr_joint_7">
-        <command_interface name="position" />
-        <command_interface name="velocity" />
-        <state_interface name="position">
-          <param name="initial_value">${radians(-135)}</param>
-        </state_interface>
-        <state_interface name="velocity">
-          <param name="initial_value">0.0</param>
-        </state_interface>
-      </joint>
     </ros2_control>
   </xacro:macro>
