Commit message: Separate grippers from base Yumi

File: robot_specific_config/abb_irb14000_support/urdf/irb14000.urdf.xacro (robot description, xacro)
@@ -10,4 +10,18 @@
   <xacro:include filename="$(find abb_irb14000_support)/urdf/irb14000_macro.xacro" />
   <xacro:irb14000 prefix="" />
+  <!-- Right gripper -->
+  <xacro:smart_gripper
+    parent="robr_tool0"
+    prefix="grpr_"
+  >
+    <origin xyz="0 0 0.007" rpy="0 0 ${radians(180)}" />
+  </xacro:smart_gripper>
+  <!-- Left gripper -->
+  <xacro:smart_gripper
+    parent="robl_tool0"
+    prefix="grpl_"
+  >
+    <origin xyz="0 0 0.007" rpy="0 0 ${radians(180)}" />
+  </xacro:smart_gripper>
   <!-- ros2_control -->
   <xacro:include filename="$(find abb_irb14000_support)/urdf/irb14000_ros2_control.xacro" />

File: robot_specific_config/abb_irb14000_support/urdf/irb14000_macro.xacro (robot description, xacro)
@@ -55,18 +55,4 @@
       <origin xyz="0.05355 0.07250 0.41492" rpy="0.9781 -0.5716 2.3180" />
     </xacro:irb14000_arm>
-    <!-- Right gripper -->
-    <xacro:smart_gripper
-      parent="${prefix}robr_tool0"
-      prefix="${prefix}grpr_"
-    >
-      <origin xyz="0 0 0.007" rpy="0 0 ${radians(180)}" />
-    </xacro:smart_gripper>
-    <!-- Left gripper -->
-    <xacro:smart_gripper
-      parent="${prefix}robl_tool0"
-      prefix="${prefix}grpl_"
-    >
-      <origin xyz="0 0 0.007" rpy="0 0 ${radians(180)}" />
-    </xacro:smart_gripper>
   </xacro:macro>
 </robot>
