Commit message: Include base_link for yumi arm

File: robot_specific_config/abb_irb14000_support/urdf/irb14000_arm_macro.xacro (robot description, xacro)
@@ -4,4 +4,5 @@
   <xacro:macro name="irb14000_arm" params="parent prefix *origin">
     <!-- Links -->
+    <link name="${prefix}base_link" />
     <link name="${prefix}link_1">
       <inertial>
@@ -152,8 +153,13 @@
     </link>
     <!-- Joints -->
+    <joint name="${prefix}base_joint" type="fixed">
+      <parent link="${parent}" />
+      <child link="${prefix}base_link" />
+      <xacro:insert_block name="origin" />
+    </joint>
     <joint name="${prefix}joint_1" type="revolute">
-      <parent link="${parent}" />
+      <parent link="${prefix}base_link" />
       <child link="${prefix}link_1" />
-      <xacro:insert_block name="origin" />
+      <origin xyz="0 0 0" rpy="0 0 0" />
       <axis xyz="0 0 1" />
       <limit lower="${radians(-168.5)}" upper="${radians(168.5)}" effort="300" velocity="${radians(180)}" />

Commit message: Update joint order to match control

File: robot_specific_config/abb_irb14000_support/urdf/irb14000_arm_macro.xacro (robot description, xacro)
@@ -174,5 +174,5 @@
       <dynamics damping="0.5" />
     </joint>
-    <joint name="${prefix}joint_7" type="revolute">
+    <joint name="${prefix}joint_3" type="revolute">
       <parent link="${prefix}link_2" />
       <child link="${prefix}link_3" />
@@ -182,5 +182,5 @@
       <dynamics damping="0.5" />
     </joint>
-    <joint name="${prefix}joint_3" type="revolute">
+    <joint name="${prefix}joint_4" type="revolute">
       <parent link="${prefix}link_3" />
       <child link="${prefix}link_4" />
@@ -190,5 +190,5 @@
       <dynamics damping="0.5" />
     </joint>
-    <joint name="${prefix}joint_4" type="revolute">
+    <joint name="${prefix}joint_5" type="revolute">
       <parent link="${prefix}link_4" />
       <child link="${prefix}link_5" />
@@ -198,5 +198,5 @@
       <dynamics damping="0.5" />
     </joint>
-    <joint name="${prefix}joint_5" type="revolute">
+    <joint name="${prefix}joint_6" type="revolute">
       <parent link="${prefix}link_5" />
       <child link="${prefix}link_6" />
@@ -206,5 +206,5 @@
       <dynamics damping="0.5" />
     </joint>
-    <joint name="${prefix}joint_6" type="revolute">
+    <joint name="${prefix}joint_7" type="revolute">
       <parent link="${prefix}link_6" />
       <child link="${prefix}link_7" />

File: robot_specific_config/abb_irb14000_support/urdf/irb14000_ros2_control.xacro (robot description, xacro)
@@ -40,5 +40,5 @@
         </state_interface>
       </joint>
-      <joint name="${prefix}robl_joint_7">
+      <joint name="${prefix}robl_joint_3">
         <command_interface name="position" />
         <command_interface name="velocity" />
@@ -50,5 +50,5 @@
         </state_interface>
       </joint>
-      <joint name="${prefix}robl_joint_3">
+      <joint name="${prefix}robl_joint_4">
         <command_interface name="position" />
         <command_interface name="velocity" />
@@ -60,5 +60,5 @@
         </state_interface>
       </joint>
-      <joint name="${prefix}robl_joint_4">
+      <joint name="${prefix}robl_joint_5">
         <command_interface name="position" />
         <command_interface name="velocity" />
@@ -70,5 +70,5 @@
         </state_interface>
       </joint>
-      <joint name="${prefix}robl_joint_5">
+      <joint name="${prefix}robl_joint_6">
         <command_interface name="position" />
         <command_interface name="velocity" />
@@ -80,5 +80,5 @@
         </state_interface>
       </joint>
-      <joint name="${prefix}robl_joint_6">
+      <joint name="${prefix}robl_joint_7">
         <command_interface name="position" />
         <command_interface name="velocity" />
@@ -110,5 +110,5 @@
         </state_interface>
       </joint>
-      <joint name="${prefix}robr_joint_7">
+      <joint name="${prefix}robr_joint_3">
         <command_interface name="position" />
         <command_interface name="velocity" />
@@ -120,5 +120,5 @@
         </state_interface>
       </joint>
-      <joint name="${prefix}robr_joint_3">
+      <joint name="${prefix}robr_joint_4">
         <command_interface name="position" />
         <command_interface name="velocity" />
@@ -130,5 +130,5 @@
         </state_interface>
       </joint>
-      <joint name="${prefix}robr_joint_4">
+      <joint name="${prefix}robr_joint_5">
         <command_interface name="position" />
         <command_interface name="velocity" />
@@ -140,5 +140,5 @@
         </state_interface>
       </joint>
-      <joint name="${prefix}robr_joint_5">
+      <joint name="${prefix}robr_joint_6">
         <command_interface name="position" />
         <command_interface name="velocity" />
@@ -150,5 +150,5 @@
         </state_interface>
       </joint>
-      <joint name="${prefix}robr_joint_6">
+      <joint name="${prefix}robr_joint_7">
         <command_interface name="position" />
         <command_interface name="velocity" />
